File: Hardware/9v_reg.kicad_sch (KiCad schematic)
At the start: 7 parts, among them U1 TPS54302

Commit message: Finalize schematic: Add connectors, LEDs, Buzzer and fix all ERC errors
Connections:
- net GND: no longer C1.1, U1.3 (VIN), U1.5 (EN)
- new net VBAT_IN: C1.1, U1.3 (VIN), U1.5 (EN)
Changed lines of the file:
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@@
-	)
-	(junction
-		(at 107.95 93.98)
-		(diameter 0)
-		(color 0 0 0 0)
 	)
 	(junction
@@
 	)
 	(junction
-		(at 111.76 91.44)
-		(diameter 0)
-		(color 0 0 0 0)
-	)
-	(junction
 		(at 129.54 101.6)
 		(diameter 0)
@@
 	(wire
 		(pts
-			(xy 107.95 91.44) (xy 107.95 93.98)
-		)
-		(stroke
-			(width 0)
-			(type default)
-		)
-	)
-	(wire
-		(pts
 			(xy 147.32 109.22) (xy 148.59 109.22)
 		)
@@
 		)
 		(stroke
-			(width 0)
-			(type default)
-		)
-	)
-	(wire
-		(pts
-			(xy 107.95 91.44) (xy 111.76 91.44)
-		)
-		(stroke

Commit message: Update schematic: Add SDIO Blackbox, ESC Redundancy and remove UART5
Changed lines of the file:
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@@
-		)
-	)
-	(label "+9V"
-		(at 124.46 93.98 0)
-		(effects
-			(font
-				(size 0.762 0.762)
-			)
-			(justify left bottom)
 		)
 	)

Commit message: Finalize component placement and silkscreen
Parts:
- C1, C2: footprint (none) -> Capacitor_SMD:C_0805_2012Metric
- C3: footprint (none) -> Capacitor_SMD:C_0402_1005Metric
- L1: footprint (none) -> Inductor_SMD:L_Taiyo-Yuden_NR-40xx
- R1, R2: footprint (none) -> Resistor_SMD:R_0402_1005Metric
Changed lines of the file:
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@@
 			)
 		)
-		(property "Footprint" ""
+		(property "Footprint" "Capacitor_SMD:C_0805_2012Metric"
 			(at 115.57 93.98 0)
 			(effects
@@
 			)
 		)
-		(property "Footprint" ""
+		(property "Footprint" "Resistor_SMD:R_0402_1005Metric"
 			(at 143.51 110.998 90)
 			(effects
@@
 			)
 		)
-		(property "Footprint" ""
+		(property "Footprint" "Capacitor_SMD:C_0402_1005Metric"
 			(at 135.89 104.14 0)
 			(effects
@@
 			)
 		)
-		(property "Footprint" ""
+		(property "Footprint" "Inductor_SMD:L_Taiyo-Yuden_NR-40xx"
 			(at 130.81 97.79 0)
 			(effects
@@
 			)
 		)
-		(property "Footprint" ""
+		(property "Footprint" "Capacitor_SMD:C_0805_2012Metric"
 			(at 121.92 93.98 0)
 			(effects
@@
 			)
 		)
-		(property "Footprint" ""
+		(property "Footprint" "Resistor_SMD:R_0402_1005Metric"
 			(at 143.51 113.792 90)
 			(effects
